Commit message: chaning back to the V13 urdf

File: assets/urdf/gogoro/urdf/scooter_V14.urdf (robot description, URDF)
Before this commit: robot gogoro_and_thormang3, 60 links, 59 joints
Links:
- link dummy_link1: mass None -> 0.00001
- link dummy_link2: mass None -> 0.00001
Joints:
- joint base_x: limit lower=-0.1 upper=0.1 effort=0.0 velocity=0.00001 -> lower=-0.1 upper=0.1 effort=0.0 velocity=1; type fixed -> prismatic
- joint base_y: limit lower=-0.1 upper=0.1 effort=0.0 velocity=0.00001 -> lower=-0.1 upper=0.1 effort=0.0 velocity=1; type fixed -> prismatic
- joint base_z: limit lower=-0.1 upper=0.1 effort=0.0 velocity=0.00001 -> lower=-0.1 upper=0.1 effort=0.0 velocity=1; type fixed -> prismatic
